File: kicad/fdshield-sop/fdshield/fdshield.kicad_pcb (KiCad board)
At the start: 2 copper layers, 68.6 x 53.3 mm, 29 parts, among them J1 Conn_02x17_Odd_Even, P1 Power, P2 Analog, P3 Digital, P4 Digital, U1 74LS74, U3 74LS08, U4 74LS125, U5 23LCxxx, U6 74HCU04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

Commit message: PCB data update (WG) (rev_h)
Parts:
- added JP5: Jumper_2_Open, Connector_PinHeader_2.54mm:PinHeader_1x02_P2.54mm_Vertical, F.Cu at (174.5, 118.1)
- moved C6 41.8 mm to (165.8, 80.6)
- moved C5 41.5 mm to (161.6, 80.6)
- moved Y1 34.8 mm to (161.3, 85.1)
- moved R7 29.7 mm to (163.7, 88.9)
- moved U3 28.0 mm to (144.0, 109.2)
- moved U6 24.5 mm to (165.0, 94.5)
- moved U5 8.64 mm to (143.4, 83.8)
- moved U4 8.64 mm to (144.0, 94.6)
- moved U1 5.81 mm to (165.0, 109.2)
- moved C4 3.59 mm to (157.2, 106.7), turned to 180 degrees
- moved C2 2.03 mm to (157.2, 92.1), turned to 180 degrees
- moved C3 1.78 mm to (136.3, 106.7), turned to 180 degrees
- moved C1 0.52 mm to (136.3, 92.1), turned to 180 degrees
Connections:
- net /10(**/SS) renamed /10(**/SS)
- net /11(**/MOSI) renamed /11(**/MOSI)
- J1 pad 2: (no net) -> unconnected-(J1-Pad2)
- J1 pad 3: (no net) -> unconnected-(J1-Pad3)
- P1 pad 1: (no net) -> unconnected-(P1-Pad1)
- P1 pad 2: (no net) -> /IOREF
- P1 pad 3: (no net) -> /Reset
- P1 pad 4: (no net) -> +3V3
- P1 pad 8: (no net) -> /Vin
- P2 pad 6: (no net) -> /WG_
- P3 pad 1: (no net) -> unconnected-(P3-Pad1)
- P3 pad 2: (no net) -> unconnected-(P3-Pad2)
- P3 pad 3: (no net) -> /AREF
- P4 pad 7: (no net) -> /1(Tx)
- P4 pad 8: (no net) -> /0(Rx)
- U1 pad 11: /RD -> Net-(U1-Pad11)
- U1 pad 6: (no net) -> unconnected-(U1-Pad6)
- U3 pad 11: (no net) -> unconnected-(U3-Pad11)
- U3 pad 8: (no net) -> unconnected-(U3-Pad8)
- U4 pad 11: (no net) -> /WD
- U4 pad 12: +5V -> /12(MISO)
- U4 pad 13: +5V -> /WG_
- U4 pad 8: (no net) -> unconnected-(U4-Pad8)
- U6 pad 1: /A1 -> /RD
- U6 pad 10: (no net) -> /CAP_CLK
- U6 pad 11: +5V -> Net-(C6-Pad1)
- U6 pad 12: (no net) -> Net-(C6-Pad1)
- U6 pad 13: +5V -> Net-(C5-Pad1)
- U6 pad 2: Net-(R6-Pad2) -> Net-(U6-Pad3)
- U6 pad 3: Net-(C5-Pad1) -> Net-(U6-Pad3)
- U6 pad 4: Net-(C6-Pad1) -> Net-(U6-Pad5)
- U6 pad 5: Net-(C6-Pad1) -> Net-(U6-Pad5)
- U6 pad 6: /CAP_CLK -> Net-(U1-Pad11)
- U6 pad 8: (no net) -> Net-(R6-Pad2)
- U6 pad 9: +5V -> /A1
Routing:
- net GND: track 160.9 -> 289.4 mm, vias 2 -> 17
- net /WG_: track 0.00 -> 64.3 mm, vias 0 -> 2
- net /WG: track 7.14 -> 63.2 mm, vias 1 -> 2
- net Net-(R6-Pad2): track 31.9 -> 76.6 mm
- net /WD: track 7.14 -> 36.9 mm, vias 1 -> 3
- net /10(**/SS): track 33.9 -> 16.7 mm
- net /4: track 67.1 -> 51.2 mm
- net +5V: track 206.2 -> 190.5 mm, vias 23 -> 17
- net /CAP_CLK: track 33.2 -> 48.0 mm
- net /A0: track 96.0 -> 82.4 mm, vias 7 -> 6
- net Net-(U1-Pad11): track 0.00 -> 12.2 mm, vias 0 -> 2
- net /A4: track 67.9 -> 77.7 mm, vias 2 -> 4
- net /13(SCK): track 35.0 -> 25.2 mm, vias 6 -> 0
- net /11(**/MOSI): track 32.0 -> 23.4 mm
- net /3(**): track 45.6 -> 51.4 mm, vias 5 -> 6
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- added copper zone on B.Cu, net (none)
- added copper zone on F.Cu, net (none)
- removed copper zone on B.Cu, net GND
- removed copper zone on F.Cu, net GND
Other:
- net class Default removed
- board text added: "DRIVE SELECT"
- board text added: "FLOPPY DISK SHIELD REV.H"
- board text added: "WRITE GATE"
- board text removed: "FLOPPY DISK SHIELD REV.C"
